Commit message: pybullet quadroit+nybble

File: data/Petoi/quadroit_v1.urdf (robot description, URDF)
Before this commit: robot quadroit_v1, 18 links, 17 joints
Links:
- removed link map

File: data/Petoi/quadv1.urdf (robot description, URDF)
Before this commit: robot quadroit_v1, 17 links, 16 joints
Links:
- link base_link: geometry collision mesh filename=meshes/base_link_torso.STL; visual mesh filename=meshes/base_link_torso.STL
- link foot_link_FL: geometry collision sphere radius=0.03; visual sphere radius=0.0
- link hip_link_FL: geometry collision mesh filename=meshes/leg_fr_hip.STL; visual mesh filename=meshes/leg_fr_hip.STL
- link shank_link_FL: geometry collision mesh filename=meshes/leg_fr_shank.STL; visual mesh filename=meshes/leg_fr_shank.STL
- link thigh_link_FL: geometry collision mesh filename=meshes/leg_fr_thigh.STL; visual mesh filename=meshes/leg_fr_thigh.STL
Joints:
- joint elbow_joint_FL: origin xyz=0.0008 0 0 rpy=1.57075 0 0 -> xyz=0.08 0 0 rpy=1.57075 0 0
- joint foot_FL: origin xyz=0.055 0 0 -> xyz=0.23 0 0
- joint hip_joint_FL: origin xyz=0.0675 0.05 0 rpy=1.57075 1.57075 1.57075 -> xyz=0.3 0.21 0 rpy=1.57075 1.57075 1.57075
- joint wrist_joint_FL: origin xyz=0.045 0 0 rpy=0 0 0 -> xyz=0.2 0 0 rpy=0 0 0

File: data/Petoi/test.urdf (robot description, URDF)
Before this commit: robot quadroit_v1, 17 links, 16 joints
Links:
- removed link foot_link_FL
- removed link foot_link_FR
- removed link foot_link_RL
- removed link foot_link_RR
- removed link hip_link_FL
- removed link hip_link_FR
- removed link hip_link_RL
- removed link hip_link_RR
- removed link shank_link_FL
- removed link shank_link_FR
- removed link shank_link_RL
- removed link shank_link_RR
- removed link thigh_link_FL
- removed link thigh_link_FR
- removed link thigh_link_RL
- removed link thigh_link_RR
- added link foot_link_lb
- added link foot_link_lf
- added link foot_link_rb
- added link foot_link_rf
- added link hip_link_lb, mass 2; collision mesh filename=meshes/leg_fr_hip.STL; visual mesh filename=meshes/leg_fr_hip.STL
- added link hip_link_lf, mass 2; collision mesh filename=meshes/leg_fr_hip.STL; visual mesh filename=meshes/leg_fr_hip.STL
- added link hip_link_rb, mass 2; collision mesh filename=meshes/leg_fr_hip.STL; visual mesh filename=meshes/leg_fr_hip.STL
- added link hip_link_rf, mass 2; collision mesh filename=meshes/leg_fr_hip.STL; visual mesh filename=meshes/leg_fr_hip.STL
- added link shank_link_lb, mass 2; collision mesh filename=meshes/leg_fr_shank.STL; visual mesh filename=meshes/leg_fr_shank.STL
- added link shank_link_lf, mass 2; collision mesh filename=meshes/leg_fr_shank.STL; visual mesh filename=meshes/leg_fr_shank.STL
- added link shank_link_rb, mass 2; collision mesh filename=meshes/leg_fr_shank.STL; visual mesh filename=meshes/leg_fr_shank.STL
- added link shank_link_rf, mass 2; collision mesh filename=meshes/leg_fr_shank.STL; visual mesh filename=meshes/leg_fr_shank.STL
- added link thigh_link_lb, mass 2; collision mesh filename=meshes/leg_fr_thigh.STL; visual mesh filename=meshes/leg_fr_thigh.STL
- added link thigh_link_lf, mass 2; collision mesh filename=meshes/leg_fr_thigh.STL; visual mesh filename=meshes/leg_fr_thigh.STL
- added link thigh_link_rb, mass 2; collision mesh filename=meshes/leg_fr_thigh.STL; visual mesh filename=meshes/leg_fr_thigh.STL
- added link thigh_link_rf, mass 2; collision mesh filename=meshes/leg_fr_thigh.STL; visual mesh filename=meshes/leg_fr_thigh.STL
- link base_link: geometry collision mesh filename=meshes/base_link_torso.STL; visual mesh filename=meshes/base_link_torso.STL
Joints:
- removed joint elbow_joint_FL
- removed joint elbow_joint_FR
- removed joint elbow_joint_RL
- removed joint elbow_joint_RR
- removed joint foot_FL
- removed joint foot_FR
- removed joint foot_RL
- removed joint foot_RR
- removed joint hip_joint_FL
- removed joint hip_joint_FR
- removed joint hip_joint_RL
- removed joint hip_joint_RR
- removed joint wrist_joint_FL
- removed joint wrist_joint_FR
- removed joint wrist_joint_RL
- removed joint wrist_joint_RR
- added joint elbow_joint_lb: type revolute, parent hip_link_lb, child thigh_link_lb, origin xyz=0.08 0 0 rpy=1.57075 0 0, axis 0 0 1, limit lower=-1.57075 upper=1.57075 effort=1000.0 velocity=0.5
- added joint elbow_joint_lf: type revolute, parent hip_link_lf, child thigh_link_lf, origin xyz=0.08 0 0 rpy=1.57075 0 0, axis 0 0 1, limit lower=-1.57075 upper=1.57075 effort=1000.0 velocity=0.5
- added joint elbow_joint_rb: type revolute, parent hip_link_rb, child thigh_link_rb, origin xyz=0.08 0 0 rpy=1.57075 0 0, axis 0 0 1, limit lower=-1.57075 upper=1.57075 effort=1000.0 velocity=0.5
- added joint elbow_joint_rf: type revolute, parent hip_link_rf, child thigh_link_rf, origin xyz=0.08 0 0 rpy=1.57075 0 0, axis 0 0 1, limit lower=-1.57075 upper=1.57075 effort=1000.0 velocity=0.5
- added joint foot_lb: type fixed, parent shank_link_lb, child foot_link_lb, origin xyz=0.23 0 0
- added joint foot_lf: type fixed, parent shank_link_lf, child foot_link_lf, origin xyz=0.23 0 0
- added joint foot_rb: type fixed, parent shank_link_rb, child foot_link_rb, origin xyz=0.23 0 0
- added joint foot_rf: type fixed, parent shank_link_rf, child foot_link_rf, origin xyz=0.23 0 0
- added joint hip_joint_lb: type revolute, parent base_link, child hip_link_lb, origin xyz=-0.3 0.21 0 rpy=1.57075 1.57075 1.57075, axis 0 0 1, limit lower=-1.57075 upper=1.57075 effort=1000.0 velocity=0.5
- added joint hip_joint_lf: type revolute, parent base_link, child hip_link_lf, origin xyz=0.3 0.21 0 rpy=1.57075 1.57075 1.57075, axis 0 0 1, limit lower=-1.57075 upper=1.57075 effort=1000.0 velocity=0.5
- added joint hip_joint_rb: type revolute, parent base_link, child hip_link_rb, origin xyz=-0.3 -0.21 0 rpy=1.57075 1.57075 1.57075, axis 0 0 1, limit lower=-1.57075 upper=1.57075 effort=1000.0 velocity=0.5
- added joint hip_joint_rf: type revolute, parent base_link, child hip_link_rf, origin xyz=0.3 -0.21 0 rpy=1.57075 1.57075 1.57075, axis 0 0 1, limit lower=-1.57075 upper=1.57075 effort=1000.0 velocity=0.5
- added joint wrist_joint_lb: type revolute, parent thigh_link_lb, child shank_link_lb, origin xyz=0.2 0 0 rpy=0 0 0, axis 0 0 1, limit lower=-1.57075 upper=1.57075 effort=1000.0 velocity=0.5
- added joint wrist_joint_lf: type revolute, parent thigh_link_lf, child shank_link_lf, origin xyz=0.2 0 0 rpy=0 0 0, axis 0 0 1, limit lower=-1.57075 upper=1.57075 effort=1000.0 velocity=0.5
- added joint wrist_joint_rb: type revolute, parent thigh_link_rb, child shank_link_rb, origin xyz=0.2 0 0 rpy=0 0 0, axis 0 0 1, limit lower=-1.57075 upper=1.57075 effort=1000.0 velocity=0.5
- added joint wrist_joint_rf: type revolute, parent thigh_link_rf, child shank_link_rf, origin xyz=0.2 0 0 rpy=0 0 0, axis 0 0 1, limit lower=-1.57075 upper=1.57075 effort=1000.0 velocity=0.5
