Commit message: quadroit running+ Nybble urdf minor updates scale

File: data/Petoi/nybble.urdf (robot description, URDF)
Before this commit: robot quadroit_v1, 17 links, 16 joints
Links:
- link base_link: mass 10 -> 0.2
- link foot_link_FL: mass 0.1 -> 0.01; geometry collision sphere radius=3e-6; visual sphere radius=3e-6
- link foot_link_FR: mass 0.1 -> 0.01; geometry collision sphere radius=3e-6; visual sphere radius=3e-6
- link foot_link_RL: mass 0.1 -> 0.01; geometry collision sphere radius=3e-6; visual sphere radius=3e-6
- link foot_link_RR: mass 0.1 -> 0.01; geometry collision sphere radius=3e-6; visual sphere radius=3e-6
- link hip_link_FL: mass 2 -> 0.001
- link hip_link_FR: mass 2 -> 0.001; geometry collision mesh filename=meshes/leg_fr_hip.STL scale=0.01 0.01 0.3; visual mesh filename=meshes/leg_fr_hip.STL scale=0.01 0.01 0.3
- link hip_link_RL: mass 2 -> 0.001; geometry collision mesh filename=meshes/leg_fr_hip.STL scale=0.01 0.01 0.3; visual mesh filename=meshes/leg_fr_hip.STL scale=0.01 0.01 0.3
- link hip_link_RR: mass 2 -> 0.001; geometry collision mesh filename=meshes/leg_fr_hip.STL scale=0.01 0.01 0.3; visual mesh filename=meshes/leg_fr_hip.STL scale=0.01 0.01 0.3
- link shank_link_FL: mass 2 -> 0.05
- link shank_link_FR: mass 2 -> 0.05; geometry collision mesh filename=meshes/leg_fr_shank.STL scale=0.239 0.239 0.239; visual mesh filename=meshes/leg_fr_shank.STL scale=0.239 0.239 0.239
- link shank_link_RL: mass 2 -> 0.05; geometry collision mesh filename=meshes/leg_fr_shank.STL scale=0.239 0.239 0.239; visual mesh filename=meshes/leg_fr_shank.STL scale=0.239 0.239 0.239
- link shank_link_RR: mass 2 -> 0.05; geometry collision mesh filename=meshes/leg_fr_shank.STL scale=0.239 0.239 0.239; visual mesh filename=meshes/leg_fr_shank.STL scale=0.239 0.239 0.239
- link thigh_link_FL: mass 2 -> 0.05
- link thigh_link_FR: mass 2 -> 0.05; geometry collision mesh filename=meshes/leg_fr_thigh.STL scale=0.225 0.225 0.225; visual mesh filename=meshes/leg_fr_thigh.STL scale=0.225 0.225 0.225
- link thigh_link_RL: mass 2 -> 0.05; geometry collision mesh filename=meshes/leg_fr_thigh.STL scale=0.225 0.225 0.225; visual mesh filename=meshes/leg_fr_thigh.STL scale=0.225 0.225 0.225
- link thigh_link_RR: mass 2 -> 0.05; geometry collision mesh filename=meshes/leg_fr_thigh.STL scale=0.225 0.225 0.225; visual mesh filename=meshes/leg_fr_thigh.STL scale=0.225 0.225 0.225
Joints:
- joint elbow_joint_FR: origin xyz=0.08 0 0 rpy=1.57075 0 0 -> xyz=0.0008 0 0 rpy=1.57075 0 0
- joint elbow_joint_RL: origin xyz=0.08 0 0 rpy=1.57075 0 0 -> xyz=0.0008 0 0 rpy=1.57075 0 0
- joint elbow_joint_RR: origin xyz=0.08 0 0 rpy=1.57075 0 0 -> xyz=0.0008 0 0 rpy=1.57075 0 0
- joint foot_FR: origin xyz=0.23 0 0 -> xyz=0.055 0 0
- joint foot_RL: origin xyz=0.23 0 0 -> xyz=0.055 0 0
- joint foot_RR: origin xyz=0.23 0 0 -> xyz=0.055 0 0
- joint hip_joint_FR: origin xyz=0.3 -0.21 0 rpy=1.57075 1.57075 1.57075 -> xyz=0.0675 -0.05 0 rpy=1.57075 1.57075 1.57075
- joint hip_joint_RL: origin xyz=-0.3 0.21 0 rpy=1.57075 1.57075 1.57075 -> xyz=-0.0675 0.05 0 rpy=1.57075 1.57075 1.57075
- joint hip_joint_RR: origin xyz=-0.3 -0.21 0 rpy=1.57075 1.57075 1.57075 -> xyz=-0.0675 -0.05 0 rpy=1.57075 1.57075 1.57075
- joint wrist_joint_FR: origin xyz=0.2 0 0 rpy=0 0 0 -> xyz=0.045 0 0 rpy=0 0 0
- joint wrist_joint_RL: origin xyz=0.2 0 0 rpy=0 0 0 -> xyz=0.045 0 0 rpy=0 0 0
- joint wrist_joint_RR: origin xyz=0.2 0 0 rpy=0 0 0 -> xyz=0.045 0 0 rpy=0 0 0

File: data/quadroit/quadv1.urdf (robot description, URDF)
Before this commit: robot quadroit_v1, 17 links, 16 joints
Links:
- link foot_link_FL: geometry collision sphere radius=0.03; visual sphere radius=0.03
- link foot_link_FR: geometry collision sphere radius=0.03; visual sphere radius=0.03
- link foot_link_RL: geometry collision sphere radius=0.03; visual sphere radius=0.03
- link foot_link_RR: geometry collision sphere radius=0.03; visual sphere radius=0.03
