Commit message: quad instincts and videos

File: data/quadroit/quadv1.urdf (robot description, URDF)
Before this commit: robot quadroit_v1, 17 links, 16 joints
Links:
- link foot_link_FL: geometry collision sphere radius=0.03; visual sphere radius=0.001
- link foot_link_FR: geometry collision sphere radius=0.03; visual sphere radius=0.001
- link foot_link_RL: geometry collision sphere radius=0.03; visual sphere radius=0.001
- link foot_link_RR: geometry collision sphere radius=0.03; visual sphere radius=0.001
